File: Hardware/Primavera_Monitor.sch (KiCad schematic (older format))
At the start: 13 parts

Commit message: Add Pi filter and diode switch to power supply
Parts:
- added C? (x4): C, symbol Device:C
- added D?: D, symbol Device:D
- added L?: L, symbol Device:L
- added U?: IFX27001TFV33, Package_TO_SOT_SMD:TO-252-3_TabPin2, symbol Regulator_Linear:IFX27001TFV33
- U?: symbol MSP-EXP432P401R:BackBoard -> Primavera_Monitor-rescue:BackBoard-MSP-EXP432P401R
- U?: symbol RTC_DS3231:RTC_DS3231_Mod -> Primavera_Monitor-rescue:RTC_DS3231_Mod-RTC_DS3231
- U? (x2): symbol MPU6050:MPU6050_Mod -> Primavera_Monitor-rescue:MPU6050_Mod-MPU6050
- U?: symbol BME280:BME280_Mod_LC -> Primavera_Monitor-rescue:BME280_Mod_LC-BME280
- U?: symbol SD_Card_Interface:SD_Card_Interface -> Primavera_Monitor-rescue:SD_Card_Interface-SD_Card_Interface
- U?: symbol OPB720b:OPB720b_mod -> Primavera_Monitor-rescue:OPB720b_mod-OPB720b
Connections:
- net labels added: +5V
- wire segments 71 -> 93

Commit message: Load improved msp-exp symbol
Parts:
- removed U?: BackBoard, symbol Primavera_Monitor-rescue:BackBoard-MSP-EXP432P401R
- added U?: BackBoard, MSP-EXP432P401R:MSP-EXP432P401R-Backboard, symbol MSP-EXP432P401R:BackBoard
Changed lines of the file:
@@
 $EndDescr
-$Comp
-L Primavera_Monitor-rescue:BackBoard-MSP-EXP432P401R U?
-U 1 1 615EADFD
-P 5450 3750
-F 0 "U?" H 4900 5000 50  0000 C CNN
-F 1 "BackBoard" H 5050 5100 50  0000 C CNN
-F 2 "" H 4850 2800 50  0001 C CNN
-F 3 "" H 4850 2800 50  0001 C CNN
-	1    5450 3750
-	1    0    0    -1
-$EndComp
 $Comp
 L Primavera_Monitor-rescue:RTC_DS3231_Mod-RTC_DS3231 U?
@@
 Wire Wire Line
 	9850 4700 9850 4850
+$Comp
+L MSP-EXP432P401R:BackBoard U?
+U 1 1 618500BC
+P 5450 3750
+F 0 "U?" H 5450 5281 50  0000 C CNN
+F 1 "BackBoard" H 5450 5190 50  0000 C CNN
+F 2 "MSP-EXP432P401R:MSP-EXP432P401R-Backboard" H 6750 2500 50  0001 C CNN
+F 3 "" H 4850 2800 50  0001 C CNN
+	1    5450 3750
+	1    0    0    -1
+$EndComp
 $EndSCHEMATC

Commit message: Add new SD Card Interface symbol to sch
Parts:
- removed U?: SD_Card_Interface, symbol Primavera_Monitor-rescue:SD_Card_Interface-SD_Card_Interface
- added U2: SD_Card_Interface, Connector_PinSocket_2.54mm:PinSocket_1x08_P2.54mm_Vertical, symbol SD_Card_Interface:SD_Card_Interface
- C1, C2: renamed from C?; footprint (none) -> Capacitor_SMD:C_1210_3225Metric
- C3, C4: renamed from C?; footprint (none) -> Capacitor_SMD:C_1206_3216Metric
- D1: renamed from D?; footprint (none) -> Diode_SMD:D_1206_3216Metric
- J1: renamed from J?; footprint (none) -> Connector_PinSocket_2.54mm:PinSocket_1x02_P2.54mm_Vertical
- L1: renamed from L?; footprint (none) -> Inductor_SMD:L_1210_3225Metric
- R1, R2, R3, R4, R5: renamed from R?; footprint (none) -> Resistor_SMD:R_1206_3216Metric
- U1: renamed from U?; footprint (none) -> Connector_PinSocket_2.54mm:PinSocket_1x03_P2.54mm_Vertical
- gave numbers to parts that had none: 6

Commit message: Add EMC protection, Long I2C and sd card on pcb
Parts:
- removed R2, R3: R, Resistor_SMD:R_1206_3216Metric, symbol Device:R
- removed U2: SD_Card_Interface, Connector_PinSocket_2.54mm:PinSocket_1x08_P2.54mm_Vertical, symbol SD_Card_Interface:SD_Card_Interface
- removed U7, U8: MPU6050_Mod, Connector_PinSocket_2.54mm:PinSocket_1x08_P2.54mm_Vertical, symbol Primavera_Monitor-rescue:MPU6050_Mod-MPU6050
- added C? (x6): C, symbol Device:C
- added C? (x4): C, Capacitor_SMD:C_1210_3225Metric, symbol Device:C
- added D? (x2): SP0502BAHT, Package_TO_SOT_SMD:SOT-23, symbol Power_Protection:SP0502BAHT
- added J? (x2): Conn_01x08, symbol Connector_Generic:Conn_01x08
- added J?: Micro_SD_Card_Det, symbol Connector:Micro_SD_Card_Det
- added L? (x2): L, Inductor_SMD:L_1210_3225Metric, symbol Device:L
- added R? (x6): R, symbol Device:R
- added R?: R, Resistor_SMD:R_1206_3216Metric, symbol Device:R
- added U? (x2): P82B715, symbol I2C_Peripherals:P82B715
Connections:
- net labels added: +3.3V, SD_DET
- wire segments 93 -> 203
Other:
- moved on the sheet: R1, U4, U6

Commit message: Add PCB design
Parts:
- removed C? (x2): C, symbol Device:C
- removed D?: SP0502BAHT, Package_TO_SOT_SMD:SOT-23, symbol Power_Protection:SP0502BAHT
- removed J?: Conn_01x08, symbol Connector_Generic:Conn_01x08
- removed R? (x2): R, symbol Device:R
- removed U?: P82B715, symbol I2C_Peripherals:P82B715
- added H1, H2, H3, H4: MountingHole, MountingHole:MountingHole_4.5mm, symbol Mechanical:MountingHole
- added R10, R11, R12, R8: R, Resistor_SMD:R_0603_1608Metric_Pad0.98x0.95mm_HandSolder, symbol Device:R
- C10, C11, C13, C9: renamed from C?; footprint (none) -> Capacitor_SMD:C_0603_1608Metric_Pad1.08x0.95mm_HandSolder
- C3, C4: footprint Capacitor_SMD:C_1206_3216Metric -> Capacitor_SMD:C_0603_1608Metric_Pad1.08x0.95mm_HandSolder
- C5, C6, C7, C8: renamed from C?; footprint Capacitor_SMD:C_1210_3225Metric -> Capacitor_SMD:C_0603_1608Metric_Pad1.08x0.95mm_HandSolder
- J2: renamed from J?; footprint (none) -> Connector_Card:microSD_HC_Hirose_DM3BT-DSF-PEJS
- J3: renamed from J?; footprint (none) -> Connector_Molex:Molex_Nano-Fit_105310-xx08_2x04_P2.50mm_Vertical
- R1, R4, R5: footprint Resistor_SMD:R_1206_3216Metric -> Resistor_SMD:R_0603_1608Metric_Pad0.98x0.95mm_HandSolder
- R2: renamed from R?; footprint Resistor_SMD:R_1206_3216Metric -> Resistor_SMD:R_0603_1608Metric_Pad0.98x0.95mm_HandSolder
- R3, R6, R7, R9: renamed from R?; footprint (none) -> Resistor_SMD:R_0603_1608Metric_Pad0.98x0.95mm_HandSolder
- U1: symbol Primavera_Monitor-rescue:OPB720b_mod-OPB720b -> OPB720b:OPB720b_mod
- U2: renamed from U?; footprint (none) -> Package_SO:SO-8_3.9x4.9mm_P1.27mm
- U4: symbol Primavera_Monitor-rescue:RTC_DS3231_Mod-RTC_DS3231 -> RTC_DS3231:RTC_DS3231_Mod
- U6: symbol Primavera_Monitor-rescue:BME280_Mod_LC-BME280 -> BME280:BME280_Mod_LC
- gave numbers to parts that had none: 3
Connections:
- net I2C_2_SCL: now also R10.1
- net I2C_2_SDA: now also R8.2
- net at D2.1 (K), R9.2, U2.2 (LX): now also R12.1, R8.1; no longer J3.4 (Pin_4)
- net at D2.2 (K), R7.2, U2.7 (Ly): now also R10.2, R11.2; no longer J3.3 (Pin_3)
- new net: J3.3 (Pin_3), R11.1
- new net: J3.4 (Pin_4), R12.2
- no-connect marks 0 -> 1

Commit message: Final Revision
Parts:
- removed C5, C6, C7, C8: C, Capacitor_SMD:C_0603_1608Metric_Pad1.08x0.95mm_HandSolder, symbol Device:C
- removed H1, H2, H3, H4: MountingHole, MountingHole:MountingHole_4.5mm, symbol Mechanical:MountingHole
- removed J3: Conn_01x08, Connector_Molex:Molex_Nano-Fit_105310-xx08_2x04_P2.50mm_Vertical, symbol Connector_Generic:Conn_01x08
- removed L2, L3: L, Inductor_SMD:L_1210_3225Metric, symbol Device:L
- removed U5: IFX27001TFV33, Package_TO_SOT_SMD:TO-252-3_TabPin2, symbol Regulator_Linear:IFX27001TFV33
- added D3: SP0502BAHT, Package_TO_SOT_SMD:SOT-23, symbol Power_Protection:SP0502BAHT
- added J3, J4: Conn_01x05, Connector_Molex:Molex_KK-254_AE-6410-05A_1x05_P2.54mm_Vertical, symbol Connector_Generic:Conn_01x05
- added J5: Conn_01x03, Connector_PinHeader_2.54mm:PinHeader_1x03_P2.54mm_Vertical, symbol Connector_Generic:Conn_01x03
- added U5: TC1262-33, Package_TO_SOT_SMD:SOT-223-3_TabPin2, symbol Regulator_Linear:TC1262-33
- J1: footprint Connector_PinSocket_2.54mm:PinSocket_1x02_P2.54mm_Vertical -> Connector_Molex:Molex_KK-254_AE-6410-02A_1x02_P2.54mm_Vertical
- U1: footprint Connector_PinSocket_2.54mm:PinSocket_1x03_P2.54mm_Vertical -> Connector_Molex:Molex_KK-254_AE-6410-03A_1x03_P2.54mm_Vertical
- U6: footprint Connector_PinSocket_2.54mm:PinSocket_1x04_P2.54mm_Vertical -> Connector_PinSocket_2.54mm:PinSocket_1x06_P2.54mm_Horizontal
Connections:
- net +3V3: now also J2.10 (DET_A), J3.1 (Pin_1), J4.1 (Pin_1), J4.5 (Pin_5), J5.1 (Pin_1), U5.3 (VO); no longer R2.1
- net +5V: now also U5.1 (VI)
- net CCR: now also U1.3 (Output), U3.30 (P3.6), D3.2 (K)
- net GND: now also J2.11 (SHIELD), R2.2, D3.3 (A), J3.2 (Pin_2), J3.5 (Pin_5), J4.2 (Pin_2), U5.2 (GND); no longer J2.9 (DET_B)
- net PWM: now also U3.40 (P3.7), J5.3 (Pin_3)
- net SD_DET: now also J2.9 (DET_B), R2.1, U3.28 (P5.0); no longer J2.10 (DET_A), R2.2, U3.23 (P3.0)
- net at U1.1 (Vcc): now also D3.1 (K), J5.2 (Pin_2)
- net at R11.1: now also J3.3 (Pin_3), J4.3 (Pin_3)
- net at R12.2: now also J3.4 (Pin_4), J4.4 (Pin_4)
- no-connect marks 1 -> 2
Other:
- moved on the sheet: C10, C11, C13, C9, D2, J2, R10, R11, R12, R2, R3, R6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

Commit message: Updated
Parts:
- added H1, H2, H3, H4: MountingHole, MountingHole:MountingHole_4mm, symbol Mechanical:MountingHole
Changed lines of the file:
@@
 Wire Wire Line
 	4300 4500 4550 4500
+$Comp
+L Mechanical:MountingHole H1
+U 1 1 61BABFEB
+P 7250 5350
+F 0 "H1" H 7350 5396 50  0000 L CNN
+F 1 "MountingHole" H 7350 5305 50  0000 L CNN
+F 2 "MountingHole:MountingHole_4mm" H 7250 5350 50  0001 C CNN
+F 3 "~" H 7250 5350 50  0001 C CNN
+	1    7250 5350
+	1    0    0    -1
+$EndComp
+$Comp
+L Mechanical:MountingHole H2
+U 1 1 61BAC28C
+P 7250 5550
+F 0 "H2" H 7350 5596 50  0000 L CNN
+F 1 "MountingHole" H 7350 5505 50  0000 L CNN
+F 2 "MountingHole:MountingHole_4mm" H 7250 5550 50  0001 C CNN
+F 3 "~" H 7250 5550 50  0001 C CNN
+	1    7250 5550
+	1    0    0    -1
+$EndComp
+$Comp
+L Mechanical:MountingHole H3
+U 1 1 61BAC4F7
+P 7250 5750
+F 0 "H3" H 7350 5796 50  0000 L CNN
+F 1 "MountingHole" H 7350 5705 50  0000 L CNN
+F 2 "MountingHole:MountingHole_4mm" H 7250 5750 50  0001 C CNN
+F 3 "~" H 7250 5750 50  0001 C CNN
+	1    7250 5750
+	1    0    0    -1
+$EndComp
+$Comp
+L Mechanical:MountingHole H4
+U 1 1 61BAC730
+P 7250 5950
+F 0 "H4" H 7350 5996 50  0000 L CNN
+F 1 "MountingHole" H 7350 5905 50  0000 L CNN
+F 2 "MountingHole:MountingHole_4mm" H 7250 5950 50  0001 C CNN
+F 3 "~" H 7250 5950 50  0001 C CNN
+	1    7250 5950
+	1    0    0    -1
+$EndComp
 $EndSCHEMATC
